Commit message: Added Friction to the Physics engine and .. built a test world to drive it in

File: description/robot.urdf.xacro (robot description, xacro)
@@ -2,3 +2,4 @@
 <robot xmlns:xacro="http://www.ros.org/wiki/xacro" name="jotham_s_mobile_bot">
     <xacro:include filename="robot_core.xacro" />
+    <xacro:include filename="gazebo_control.xacro" />
 </robot>

File: description/robot_core.xacro (robot description, xacro)
@@ -47,4 +47,9 @@
         </xacro:inertial_box>
     </link>
+    <gazebo reference="chassis">
+        <material>
+            Gazebo/Orange
+        </material>
+    </gazebo>
     <!--LEFT
     WHEEL LINK-->
@@ -71,4 +76,9 @@
         </xacro:inertial_cylinder>
     </link>
+    <gazebo reference="left_wheel">
+        <material>
+            Gazebo/Blue
+        </material>
+    </gazebo>
     <!--RIGHT
     WHEEL LINK-->
@@ -95,4 +105,9 @@
         </xacro:inertial_cylinder>
     </link>
+    <gazebo reference="right_wheel">
+        <material>
+            Gazebo/Blue
+        </material>
+    </gazebo>
     <!-- CASTER WHEEL LINK -->
     <joint name="caster_wheel_joint" type="fixed">
@@ -117,3 +132,10 @@
         </xacro:inertial_sphere>
     </link>
+    <gazebo reference="caster_wheel">
+        <material>
+            Gazebo/Black
+        </material>
+        <mu1 value="0.001" />
+        <mu2 value="0.001" />
+    </gazebo>
 </robot>
