Commit message: Implemented localization using AMCL  with NAV2 and slam_toolbox

File: description/robot_core.xacro (robot description, xacro)
@@ -20,4 +20,11 @@
     LINK-->
     <link name="base_link" />
+    <!-- BASE_FOOTPRINT LINK-->
+    <joint name="base_footprint_joint" type="fixed">
+        <parent link="base_link" />
+        <child link="base_footprint" />
+        <origin xyz="0 0 0" rpy="0 0 0" />
+    </joint>
+    <link name="base_footprint" />
     <!--CHASSIS
     JOINT-->
