Commit message: Implemented ball detection and tracking

File: description/camera.xacro (robot description, xacro)
@@ -4,5 +4,5 @@
         <parent link="chassis" />
         <child link="camera_link" />
-        <origin xyz="0.305 0 0.08" rpy="0 0 0" />
+        <origin xyz="0.305 0 0.08" rpy="0 0.18 0" />
     </joint>
     <link name="camera_link">
